File: Flyback/pcb/Flyback_Layout_1.kicad_pcb (KiCad board)
At the start: 2 copper layers, 34 parts

Commit message: layout ...
Parts:
- added C_compP1: C, Capacitors_THT:CP_Radial_D10.0mm_P2.50mm, F.Cu at (135.3, 64.1)
- added R_OPTO_colector1: R, Resistors_THT:R_Axial_DIN0204_L3.6mm_D1.6mm_P7.62mm_Horizontal, F.Cu at (137.8, 88.3)
- added Rgate1: R, Resistors_THT:R_Axial_DIN0204_L3.6mm_D1.6mm_P7.62mm_Horizontal, F.Cu at (146.7, 104.8)
- moved R_CS1 376.0 mm to (139.7, 132.1), turned to 90 degrees
- moved Dsnub1 366.3 mm to (151.1, 120.0), turned to 270 degrees
- moved C_VCC1 345.5 mm to (118.7, 86.4), turned to 270 degrees
- moved RT1 340.5 mm to (123.8, 84.5), turned to 90 degrees
- moved CT1 339.2 mm to (114.9, 80.0), turned to 270 degrees
- moved R_compP1 332.0 mm to (132.7, 76.8)
- moved R_mininalLOAD1 300.9 mm to (200.7, 82.5)
- moved C_CSF1 300.2 mm to (120.7, 80.6), turned to 180 degrees
- moved D_VCC1 296.0 mm to (135.9, 92.1)
- moved Rsnub1 295.2 mm to (151.1, 109.9), turned to 270 degrees
- moved Rtrafo1 286.6 mm to (158.8, 92.1), turned to 180 degrees
- moved R_FGB1 272.8 mm to (132.7, 71.1)
- moved U_OPTO1 272.2 mm to (158.8, 84.5), turned to 180 degrees
- moved R_compZ1 270.5 mm to (170.2, 73.7)
- moved D_OUT1 264.9 mm to (201.9, 92.7)
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Connections:
- U_OPTO1 pad 3: (no net) -> Net-(R_FGB1-Pad2)
- U_OPTO1 pad 4: (no net) -> Net-(R_OPTO_colector1-Pad2)
Routing:
- net GND: track 85.1 -> 137.8 mm
- net ISENSE: track 0.00 -> 45.1 mm
- net Net-(Q_NMOS1-Pad3): track 0.00 -> 26.7 mm
- net GATE: track 0.00 -> 24.0 mm
- net VCC: track 15.5 -> 33.3 mm
- net COMP: track 0.00 -> 16.4 mm
- net RTCT: track 0.00 -> 15.6 mm
- net VREF: track 0.00 -> 15.5 mm
- net Net-(R_FGB1-Pad2): track 0.00 -> 15.3 mm
- net VRET: track 54.7 -> 67.4 mm
- net VFB: track 0.00 -> 11.4 mm
- net Net-(Csnub1-Pad2): track 0.00 -> 10.5 mm
- net Net-(R_OPTO_colector1-Pad2): track 0.00 -> 7.29 mm
- net OUTPUT: track 25.6 -> 32.0 mm
- net DRENO: track 0.00 -> 4.49 mm
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
Commit message: git add img/!
Parts:
- added C_compZ1: C, Capacitors_THT:CP_Radial_D10.0mm_P2.50mm, F.Cu at (170.2, 61.5)
- added C_em1: C, Capacitors_THT:C_Rect_L18.0mm_W9.0mm_P15.00mm_FKS3_FKP3, F.Cu at (62.4, 98.7)
- added C_em2: C, Capacitors_THT:C_Rect_L18.0mm_W9.0mm_P15.00mm_FKS3_FKP3, F.Cu at (81.4, 98.7)
- added D_Zener_OUT1: 12V, Diodes_THT:D_DO-35_SOD27_P7.62mm_Horizontal, F.Cu at (245.8, 141.9)
- added RZD_OUT1: R, Resistors_THT:R_Axial_DIN0204_L3.6mm_D1.6mm_P7.62mm_Horizontal, F.Cu at (234.6, 119.7)
- added RZD_VCC1: R, Resistors_THT:R_Axial_DIN0204_L3.6mm_D1.6mm_P7.62mm_Horizontal, F.Cu at (256.8, 130.0)
- C_OUT1: footprint Capacitors_THT:CP_Radial_D4.0mm_P1.50mm -> Capacitors_THT:CP_Radial_D10.0mm_P5.00mm
- C_in1: value 2200uF -> 150uF
- Csnub1: footprint Capacitors_THT:CP_Radial_D4.0mm_P1.50mm -> Capacitors_THT:C_Rect_L24.0mm_W12.2mm_P22.50mm_MKT
- Rsnub1: footprint Resistors_THT:R_Axial_DIN0204_L3.6mm_D1.6mm_P7.62mm_Horizontal -> Resistors_THT:R_Axial_Power_L20.0mm_W6.4mm_P22.40mm
- moved Csnub1 81.6 mm to (176.1, 30.9), turned to 0 degrees
- moved R_FBB1 50.0 mm to (177.9, 117.5)
- moved C_OUT1 27.6 mm to (178.4, 87.7), turned to 270 degrees
- moved Rsnub1 11.2 mm to (162.4, 109.7)
- moved D_OUT1 8.86 mm to (200.2, 84.0)
- moved R_mininalLOAD1 8.78 mm to (197.7, 90.8), turned to 270 degrees
- moved R_TLbias1 6.11 mm to (170.4, 78.7)
- moved R_LED1 3.86 mm to (170.4, 87.7)
- moved C_in1 0.10 mm to (114.9, 111.2)
Connections:
- C_OUT1 pad 2: GND -> GOUT
- R_FBB1 pad 1: GND -> GOUT
- R_TLbias1 pad 2: Net-(C_compZ1-Pad2) -> Net-(C_compZ1-Pad1)
- R_mininalLOAD1 pad 2: GND -> GOUT
- U_OPTO1 pad 2: Net-(C_compZ1-Pad2) -> Net-(C_compZ1-Pad1)
Routing:
- net Net-(Csnub1-Pad2): track 10.5 -> 27.2 mm
- net VRET: track 67.4 -> 74.3 mm
- net Net-(C_em2-Pad2): track 24.3 -> 17.7 mm
- net Net-(C_em2-Pad1): track 24.3 -> 17.8 mm

Commit message: footprit ...
Parts:
- added Trafo1: Transformer_1P_2S, core_transformer_THT:core_30-7, F.Cu at (184.9, 106.8)
- C_compP1, C_compZ1: footprint Capacitors_THT:CP_Radial_D10.0mm_P2.50mm -> Capacitors_THT:C_Axial_L3.8mm_D2.6mm_P7.50mm_Horizontal
- Csnub1: footprint Capacitors_THT:C_Rect_L24.0mm_W12.2mm_P22.50mm_MKT -> Capacitors_THT:C_Rect_L24.0mm_W7.0mm_P22.50mm_MKT
- moved RZD_VCC1 129.1 mm to (132.7, 94.3), turned to 180 degrees
- moved D_Zener_OUT1 117.5 mm to (136.2, 99.5)
- moved RZD_OUT1 106.3 mm to (130.8, 96.8)
- moved Csnub1 81.7 mm to (155.5, 110.0), turned to 270 degrees
- moved C_OUT1 37.9 mm to (214.0, 100.6)
- moved R_FBU1 31.5 mm to (210.5, 92.7), turned to 0 degrees
- moved R_FBB1 31.5 mm to (206.7, 105.0), turned to 90 degrees
- moved R_compZ1 31.2 mm to (199.5, 84.2)
- moved C_compZ1 29.6 mm to (196.9, 74.2), turned to 270 degrees
- moved R_mininalLOAD1 29.1 mm to (226.7, 92.8)
- moved Dsnub1 23.4 mm to (167.9, 136.3), turned to 180 degrees
- moved R_TLbias1 22.7 mm to (192.8, 81.8), turned to 90 degrees
- moved R_LED1 21.2 mm to (188.2, 76.3)
- moved U_OPTO1 19.1 mm to (176.1, 76.3)
- moved D_OUT1 12.2 mm to (202.4, 96.1), turned to 270 degrees
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Routing:
- net GND: track 137.8 -> 458.9 mm
- net VOUT: track 0.00 -> 65.2 mm
- net DRENO: track 4.49 -> 54.2 mm
- net GOUT: track 0.00 -> 37.3 mm
- net Net-(R_OPTO_colector1-Pad2): track 7.29 -> 33.7 mm
- net Net-(Rtrafo1-Pad1): track 0.00 -> 23.5 mm
- net Net-(C_compZ1-Pad1): track 0.00 -> 21.0 mm
- net Net-(R_FBB1-Pad2): track 0.00 -> 19.3 mm
- net VRET: track 74.3 -> 88.7 mm
- net Net-(Csnub1-Pad2): track 27.2 -> 14.1 mm
- net Net-(R_FGB1-Pad2): track 15.3 -> 28.0 mm
- net Vtrafo: track 0.00 -> 7.50 mm
- net VFB: track 11.4 -> 17.6 mm
- net Net-(R_LED1-Pad2): track 0.00 -> 4.53 mm
- net Net-(D_Zener_OUT1-Pad1): track 0.00 -> 3.93 mm
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
Commit message: add photo
Parts:
- added L_em1: L, Inductors_THT:L_Axial_L14.0mm_D4.5mm_P15.24mm_Horizontal_Fastron_LACC, F.Cu at (75.4, 196.3)
- added L_em2: L, Inductors_THT:L_Axial_L14.0mm_D4.5mm_P15.24mm_Horizontal_Fastron_LACC, F.Cu at (105.9, 196.3)
- added Pin_gout1: CONN_01X01, Connectors:Pin_d1.4mm_L8.5mm_W2.8mm_FlatFork, F.Cu at (139.7, 74.8)
- added Pin_in_neg1: CONN_01X01, Connectors:Pin_d1.4mm_L8.5mm_W2.8mm_FlatFork, F.Cu at (139.9, 185.3)
- added Pin_in_pos1: CONN_01X01, Connectors:Pin_d1.4mm_L8.5mm_W2.8mm_FlatFork, F.Cu at (139.9, 181.5)
- added Pin_vout1: CONN_01X01, Connectors:Pin_d1.4mm_L8.5mm_W2.8mm_FlatFork, F.Cu at (139.7, 71.0)
- added TL1: Ajus_Shunt, TO_SOT_Packages_THT:TO-92_Inline_Wide, F.Cu at (80.0, 70.2)
- moved R_mininalLOAD1 120.1 mm to (110.7, 62.0), turned to 0 degrees
- moved C_compZ1 116.9 mm to (80.0, 75.6), turned to 0 degrees
- moved R_FBU1 116.1 mm to (98.5, 62.0)
- moved R_compZ1 110.0 mm to (90.0, 73.0), turned to 90 degrees
- moved R_LED1 106.4 mm to (82.1, 84.3), turned to 270 degrees
- moved R_TLbias1 105.2 mm to (87.7, 79.7), turned to 180 degrees
- moved D_OUT1 103.8 mm to (101.9, 70.1), turned to 0 degrees
- moved R_FBB1 103.6 mm to (110.8, 65.8), turned to 180 degrees
- moved U_OPTO1 96.0 mm to (82.2, 96.5), turned to 270 degrees
- moved C_em1 94.7 mm to (83.3, 191.0), turned to 0 degrees
- moved C_compP1 93.0 mm to (73.4, 135.5), turned to 270 degrees
- moved R_FGB1 86.1 mm to (78.6, 139.9), turned to 90 degrees
- moved R_OPTO1 84.5 mm to (79.5, 129.6), turned to 0 degrees
- moved Dret_1 83.2 mm to (75.5, 172.8), turned to 0 degrees
- moved CT1 82.8 mm to (85.9, 157.6), turned to 0 degrees
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Routing:
- net GOUT: track 37.3 -> 167.8 mm
- net Net-(C_em1-Pad1): track 0.00 -> 98.8 mm
- net VRET: track 88.7 -> 152.7 mm
- net Net-(C_em1-Pad2): track 0.00 -> 48.4 mm
- net GND: track 458.9 -> 499.2 mm
- net Net-(C_compZ1-Pad1): track 21.0 -> 52.8 mm
- net Net-(R_FBB1-Pad2): track 19.3 -> 46.7 mm
- net Net-(R_FGB1-Pad2): track 28.0 -> 53.6 mm
- net VOUT: track 65.2 -> 89.8 mm
- net ISENSE: track 45.1 -> 60.9 mm
- net VCC: track 33.3 -> 48.3 mm
- net Net-(C_em2-Pad1): track 17.8 -> 25.8 mm
- net Net-(C_em2-Pad2): track 17.7 -> 25.3 mm
- net DRENO: track 54.2 -> 60.5 mm
- net Net-(Q_NMOS1-Pad3): track 26.7 -> 32.5 mm
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Other:
- board outline added: 101.6 x 142.1 mm
- net class Default: trace_width 0.5 -> 1
